File: pcb/display_oled.kicad_sch (KiCad schematic)
At the start: 4 parts, among them J1 Molex-50511, Q1 AO3413, U1 SSD1306

Commit message: Use KiCad SOT-23-3 footprint
The copied footprint was likely due to a missing 3D model, but the
current KiCad library has a 3D model now.
Parts:
- Q1: footprint keyboard:SOT-23-3 -> Package_TO_SOT_SMD:SOT-23-3
Changed lines of the file:
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@@
 			)
 		)
-		(property "Footprint" "keyboard:SOT-23-3"
+		(property "Footprint" "Package_TO_SOT_SMD:SOT-23-3"
 			(at 121.92 55.88 0)
 			(effects
