File: pcb/peripheral.kicad_sch (KiCad schematic)
At the start: 0 parts

Commit message: Add Molex connector to peripheral template
Parts:
- added J1: Molex-50511, keyboard:Molex_5051100692_1x06_P0.5mm_Anchor_2, symbol Connector_Generic:Conn_01x06
Connections:
- new net DATA1: J1.3 (Pin_3)
- new net DATA2: J1.4 (Pin_4)
- new net DATA3: J1.5 (Pin_5)
- new net GND: J1.1 (Pin_1), J1.6 (Pin_6)
- new net VDD: J1.2 (Pin_2)
