File: pcb/numpad.kicad_pcb (KiCad board)
At the start: 2 copper layers, 76.2 x 123.5 mm, 85 parts, among them J1 HRO_TYPE-C-31-M-12, J2 Molex-505110, J3 Molex-Pico-EZMate, J4 JST-SH, J5 JTAG, SW1 F1, SW10 8, SW11 9, SW12 4, SW13 5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

Commit message: Fix BOM and update DRC exclusions
Parts:
- U1: value MDBT50Q-1MV2 -> MDBT50Q-P1MV2
